Commit message: added teleop 4WS working sim

File: src/scouting_robot_description/urdf/base.urdf.xacro (robot description, xacro)
@@ -5,7 +5,8 @@
 		<link name="base_link">
 		   	<inertial>
-				<origin xyz="0 0.00163 0.07094" rpy="0 0 0" />
+				<origin xyz="-0.20 0.00163 0.07094" rpy="0 0 0" />
 				<mass value="1.5" />
 				<inertia ixx="0.0025" ixy="0.00013" ixz="0.00419" iyy="0.01593" iyz="0" izz="0.01605" />
+				<gravity>1</gravity>
 			</inertial>
 			<visual>
@@ -48,6 +49,12 @@
 			<child  link="back_link"/>
 			<axis xyz="1 0 0"/>
-			<limit lower="-1.5" upper="1.5" effort="10" velocity="5"/>
+			<limit lower="-${M_PI*0.25}" upper="${M_PI*0.25}" effort="10" velocity="5"/>
 		</joint>
+		<gazebo reference="base_link">
+			<selfCollide>false</selfCollide>
+		</gazebo>
+		<gazebo reference="back_link">
+			<selfCollide>false</selfCollide>
+		</gazebo>
 	</xacro:macro>
 </robot>

File: src/scouting_robot_description/urdf/scouting_robot.urdf.xacro (robot description, xacro)
@@ -17,11 +17,12 @@
   <xacro:include filename="wheels.urdf.xacro" />
   <xacro:base colour="silver"/>
-	<xacro:wheel name="front_left"  parent="base_link" right="1"  front="1" />
-	<xacro:wheel name="front_right" parent="base_link" right="-1" front="1" />
-	<xacro:wheel name="back_left"   parent="back_link" right="1"  front="-1" />
-	<xacro:wheel name="back_right"  parent="back_link" right="-1" front="-1" />
+	<xacro:wheel name="front_left"  parent="base_link" left="1"  front="1" />
+	<xacro:wheel name="front_right" parent="base_link" left="-1" front="1" />
+	<xacro:wheel name="back_left"   parent="back_link" left="1"  front="-1" />
+	<xacro:wheel name="back_right"  parent="back_link" left="-1" front="-1" />
   <gazebo>
     <plugin name="gazebo_ros_control" filename="libgazebo_ros_control.so">
       <robotNamespace>/</robotNamespace>
+      <robotSimType>gazebo_ros_control/DefaultRobotHWSim</robotSimType>
     </plugin>
   </gazebo>

File: src/scouting_robot_description/urdf/wheels.urdf.xacro (robot description, xacro)
@@ -14,14 +14,14 @@
 	<xacro:property name="wheel_Ixx_Iyy" value="${wheel_mass*(3*(wheel_radius**2 + wheel_inner_radius**2) + wheel_length**2)/12}" />
 	<xacro:property name="wheel_Izz" value="${wheel_mass*(wheel_radius**2 + wheel_inner_radius**2)/2}" />
-	<xacro:macro name="wheel" params="name parent right front">
+	<xacro:macro name="wheel" params="name parent left front">
 		<link name="${name}_ankle">
 			<inertial>
-				<!-- from Solid Edge "Steering Block.asm" -->
 				<origin xyz="0 0.019 -0.0325" rpy="0 0 0" />
 				<mass value="0.271" />
 				<inertia ixx="0.01" iyy="0.01" izz="0.01" ixy="0" ixz="0" iyz="0" />
+				<gravity>1</gravity>
 			</inertial>
 			<visual>
-				<origin xyz="0 0 0" rpy="0 0 ${M_PI if right == -1 else 0}"/>
+				<origin xyz="0 0 0" rpy="0 0 ${M_PI if left == -1 else 0}"/>
 				<geometry>
 					<mesh filename="package://scouting_robot_description/meshes/hub.dae" />
@@ -30,5 +30,5 @@
 			</visual>
 			<collision>
-				<origin xyz="0 0 0" rpy="0 0 ${M_PI if right == -1 else 0}"/>
+				<origin xyz="0 0 0" rpy="0 0 ${M_PI if left == -1 else 0}"/>
 				<geometry>
 					<mesh filename="package://scouting_robot_description/meshes/hub.dae" />
@@ -45,14 +45,15 @@
 				<mass value="1.24" />
 				<inertia ixx="${wheel_Ixx_Iyy}" iyy="${wheel_Ixx_Iyy}"  izz="${wheel_Izz}" ixy="0.0" ixz="0.0" iyz="0.0" />
+				<gravity>1</gravity>
 			</inertial>
 			<visual>
-				<xacro:if value="${right == -1}">
+				<xacro:if value="${left == -1}">
 					<origin rpy="0 0 ${M_PI}" />
 				</xacro:if>
 				<geometry>
-					<xacro:if value="${right == 1}">
+					<xacro:if value="${left == -1}">
 						<mesh filename="package://scouting_robot_description/meshes/r_wheel.dae"/>
 					</xacro:if>
-					<xacro:if value="${right == -1}">
+					<xacro:if value="${left == 1}">
 						<mesh filename="package://scouting_robot_description/meshes/l_wheel.dae"/>
 					</xacro:if>
@@ -66,45 +67,43 @@
 			</collision>
 		</link>
-		<!-- Steering with transmissions for gazebo -->
-    <joint name="${name}_steering_joint" type="revolute">
-      <parent link="${parent}" />
-      <child link="${name}_ankle" />
-      <axis xyz="0 0 1" />
-      <origin xyz="0 ${right*ankle_offset_y} -${ankle_offset_z}" />
-      <limit lower="-${angle_limit_ccw}" upper="${angle_limit_cw}" effort="7" velocity="15" />
-      <!-- guesses -->
-    </joint>
-	 <joint name="${name}_wheel_joint" type="continuous">
-      <parent link="${name}_ankle" />
-      <child link="${name}_wheel" />
-      <axis xyz="0 1 0" />
-      <origin xyz="0 ${right*wheel_offset_y} -${wheel_offset_z}" />
-    </joint>
-<!--
-    <transmission name="${name}_steering_trans" type="SimpleTransmission">
+		<gazebo reference="${name}_wheel">
+			<selfCollide>false</selfCollide>
+		</gazebo>
+			Steering with transmissions for gazebo
+		<joint name="${name}_steering_joint" type="revolute">
+			<parent link="${parent}" />
+			<child link="${name}_ankle" />
+			<axis xyz="0 0 1" />
+			<origin xyz="0 ${left*ankle_offset_y} -${ankle_offset_z}" />
+			<limit lower="-${angle_limit_ccw}" upper="${angle_limit_cw}" effort="7" velocity="15" />
+		<!-- guesses -->
+		</joint>
+		<joint name="${name}_wheel_joint" type="continuous">
+			<parent link="${name}_ankle" />
+			<child link="${name}_wheel" />
+			<axis xyz="0 1 0" />
+			<origin xyz="0 ${left*wheel_offset_y} -${wheel_offset_z}" />
+			<limit effort="10" velocity="5"/>
+		</joint>
+<!--  -->
+		<transmission name="${name}_steering_trans">
 			<type>transmission_interface/SimpleTransmission</type>
-      <actuator name="${name}_steering_motor">
-        <hardwareInterface>PositionJointInterface</hardwareInterface>
-        <mechanicalReduction>1</mechanicalReduction>
-      </actuator>
 			<joint name="${name}_steering_joint">
 				<hardwareInterface>hardware_interface/PositionJointInterface</hardwareInterface>
 			</joint>
+			<actuator name="${name}_steering_motor" >
+				<hardwareInterface>PositionJointInterface</hardwareInterface>
+				<mechanicalReduction>1</mechanicalReduction>
+			</actuator>
 		</transmission>
--->
-    <!-- Power wheels -->
-    <transmission name="${name}_wheel_transmission" type="SimpleTransmission">
+  		<transmission name="${name}_wheel_transmission">
 			<type>transmission_interface/SimpleTransmission</type>
-			<actuator name="${name}_wheel_motor" />
 			<joint name="${name}_wheel_joint">
 				<hardwareInterface>hardware_interface/VelocityJointInterface</hardwareInterface>
 			</joint>
-		</transmission>
-  <transmission name="${name}_steering_trans" type="SimpleTransmission">
-			<type>transmission_interface/SimpleTransmission</type>
-			<actuator name="${name}_steering_motor" />
-			<joint name="${name}_steering_joint">
-				<hardwareInterface>hardware_interface/PositionJointInterface</hardwareInterface>
-			</joint>
+			<actuator name="${name}_wheel_motor" >
+				<hardwareInterface>VelocityJointInterface</hardwareInterface>
+				<mechanicalReduction>1</mechanicalReduction>
+			</actuator>
 		</transmission>
 	</xacro:macro>

Commit message: updated args and param links

File: src/scouting_robot_description/urdf/base.urdf.xacro (robot description, xacro)
@@ -1,5 +1,5 @@
 <?xml version="1.0" encoding="UTF-8"?>
 <robot xmlns:xacro="http://www.ros.org/wiki/xacro">
-	<xacro:property name="wheelbase" value="0.45" />
+	<xacro:property name="wheelbase" value="$(arg wheel_base)" />
 	<xacro:macro name="base" params="colour">
 		<link name="base_link">

File: src/scouting_robot_description/urdf/scouting_robot.urdf.xacro (robot description, xacro)
@@ -1,5 +1,5 @@
 <?xml version="1.0" encoding="UTF-8"?>
 <robot xmlns:xacro="http://www.ros.org/wiki/xacro" name="scouting_robot">
-  <xacro:property name="M_PI" value="3.1415926535897931" />
+	<xacro:property name="M_PI" value="3.1415926535897931" />
   <!-- measured mass of tyre and hub outer part: 1.238g -->
   <!-- measured mass of base block and two steering blocks: 1550 g -->

File: src/scouting_robot_description/urdf/wheels.urdf.xacro (robot description, xacro)
@@ -1,14 +1,14 @@
 <?xml version="1.0" encoding="UTF-8"?>
 <robot xmlns:xacro="http://www.ros.org/wiki/xacro">
-	<xacro:property name="angle_limit_cw" value="${M_PI/4}" />
+	<xacro:property name="angle_limit_cw"  value="${M_PI/4}" />
 	<xacro:property name="angle_limit_ccw" value="${M_PI/4}" />
-	<xacro:property name="ankle_offset_y" value="0.085" />
-	<xacro:property name="ankle_offset_z" value="0.0015" />
-	<xacro:property name="wheel_offset_y" value="0.06" />
-	<xacro:property name="wheel_offset_z" value="0.05" />
-	<xacro:property name="wheel_radius" value=".12" />
-	<xacro:property name="wheel_inner_radius" value=".045" />
-	<xacro:property name="wheel_length" value=".07" />
-	<xacro:property name="wheel_mass" value="1.24" />
+	<xacro:property name="ankle_offset_y" value="$(arg ankle_offset_y)" />
+	<xacro:property name="ankle_offset_z" value="$(arg ankle_offset_z)" />
+	<xacro:property name="wheel_offset_y" value="$(arg wheel_offset_y)" />
+	<xacro:property name="wheel_offset_z" value="$(arg wheel_offset_z)" />
+	<xacro:property name="wheel_radius" 		value="$(arg wheel_radius)" />
+	<xacro:property name="wheel_inner_radius" 	value="$(arg wheel_inner_radius)" />
+	<xacro:property name="wheel_length" value="$(arg wheel_length)" />
+	<xacro:property name="wheel_mass" 	value="$(arg wheel_mass)" />
 	<!-- from standard equation for thick-walled cylinder -->
 	<xacro:property name="wheel_Ixx_Iyy" value="${wheel_mass*(3*(wheel_radius**2 + wheel_inner_radius**2) + wheel_length**2)/12}" />

Commit message: added crabsteering

File: src/scouting_robot_description/urdf/base.urdf.xacro (robot description, xacro)
@@ -6,5 +6,5 @@
 		   	<inertial>
 				<origin xyz="-0.20 0.00163 0.07094" rpy="0 0 0" />
-				<mass value="1.5" />
+				<mass value="5" />
 				<inertia ixx="0.0025" ixy="0.00013" ixz="0.00419" iyy="0.01593" iyz="0" izz="0.01605" />
 				<gravity>1</gravity>

File: src/scouting_robot_description/urdf/wheels.urdf.xacro (robot description, xacro)
@@ -18,5 +18,5 @@
 			<inertial>
 				<origin xyz="0 0.019 -0.0325" rpy="0 0 0" />
-				<mass value="0.271" />
+				<mass value="0.4" />
 				<inertia ixx="0.01" iyy="0.01" izz="0.01" ixy="0" ixz="0" iyz="0" />
 				<gravity>1</gravity>
